Commit message: new gazebo

File: description/camera.xacro (robot description, xacro)
@@ -4,5 +4,5 @@
         <parent link="chassis"/>
         <child link="camera_link"/>
-        <origin xyz="0.150 0 0.06" rpy="0 0 0"/>
+        <origin xyz="0.190 0 0.06" rpy="0 0 0"/>
     </joint>
     <link name="camera_link">
@@ -11,5 +11,5 @@
                 <box size="0.010 0.03 0.03"/>
             </geometry>
-            <material name="green"/>
+            <material name="red"/>
         </visual>
     </link>
@@ -20,6 +20,6 @@
     </joint>
     <link name="camera_link_optical"></link>
-    <gazebo reference="camera_link">
-        <material>Gazebo/Green</material>
+     <gazebo reference="camera_link">
+        <material>Gazebo/Black</material>
         <sensor name="camera" type="camera">
             <pose> 0 0 0 0 0 0 </pose>
@@ -27,4 +27,5 @@
             <update_rate>10</update_rate>
             <camera>
+                <camera_info_topic>camera/camera_info</camera_info_topic>
                 <horizontal_fov>1.089</horizontal_fov>
                 <image>
@@ -38,7 +39,6 @@
                 </clip>
             </camera>
-            <plugin name="camera_controller" filename="libgazebo_ros_camera.so">
-                <frame_name>camera_link_optical</frame_name>
-            </plugin>
+            <topic>camera/image_raw</topic>
+            <gz_frame_id>camera_link_optical</gz_frame_id>
         </sensor>
     </gazebo>

File: description/ros2_control.xacro (robot description, xacro)
@@ -32,7 +32,7 @@
     </xacro:unless>
     <xacro:if value="$(arg sim_mode)">
-        <ros2_control name="GazeboSystem" type="system">
+        <ros2_control name="IgnitionSystem" type="system">
             <hardware>
-                <plugin>gazebo_ros2_control/GazeboSystem</plugin>
+                <plugin>ign_ros2_control/IgnitionSystem</plugin>
             </hardware>
             <joint name="left_wheel_joint">
@@ -55,5 +55,5 @@
     </xacro:if>
     <gazebo>
-        <plugin name="gazebo_ros2_control" filename="libgazebo_ros2_control.so">
+         <plugin filename="libign_ros2_control-system.so" name="ign_ros2_control::IgnitionROS2ControlPlugin">
             <parameters>$(find robotek)/config/my_controllers.yaml</parameters>
             <parameters>$(find robotek)/config/gaz_ros2_ctl_use_sim.yaml</parameters>
