Commit message: zmeny

File: description/lidar.xacro (robot description, xacro)
@@ -5,5 +5,4 @@
         <child link="laser_frame"/>
         <origin xyz="0.045 0 0.1" rpy="0 0 0"/>
-        <!-- <origin xyz="0.122 0 0.212" rpy="0 0 0"/> -->
     </joint>
     <link name="laser_frame">

File: description/robot_main.xacro (robot description, xacro)
@@ -1,5 +1,4 @@
 <?xml version="1.0"?>
 <robot xmlns:xacro="http://www.ros.org/wiki/xacro"  name="robot">
-    <xacro:arg name="use_ros2_control" default="true"/>
     <xacro:arg name="sim_mode" default="false"/>
     <!--URDF zakladny robota -->
@@ -11,9 +10,4 @@
     <!--podminka pro vyuziti ros2_control nebo gazebo_control-->
     <!--knihovny pro popis a reseni pohybu simulovaneho nebo realneho robota-->
-    <xacro:if value="$(arg use_ros2_control)">
-        <xacro:include filename="ros2_control.xacro" />
-    </xacro:if>
-    <xacro:unless value="$(arg use_ros2_control)">
-        <xacro:include filename="gazebo_control.xacro" />
-    </xacro:unless>
+    <xacro:include filename="ros2_control.xacro" />
 </robot>

File: description/ros2_control.xacro (robot description, xacro)
@@ -32,9 +32,12 @@
         </ros2_control>
     </xacro:unless>
-    <xacro:unless value="$(arg sim_mode)">
+    <xacro:if value="$(arg sim_mode)">
+    <!--resource manager gazebo ignition / kontroluje akcni cleny po hardwarove strance -->
         <ros2_control name="IgnitionSystem" type="system">
             <hardware>
+                <!--hardwarove rozhrani plugin-->
                 <plugin>ign_ros2_control/IgnitionSystem</plugin>
             </hardware>
+                <!--kloub robota dle  URDF-->
             <joint name="left_wheel_joint">
                 <command_interface name="velocity">
@@ -55,8 +58,10 @@
         </ros2_control>
     </xacro:if>
+    <!--spusteni controller manager a simulace hardware -->
     <gazebo>
          <plugin filename="libign_ros2_control-system.so" name="ign_ros2_control::IgnitionROS2ControlPlugin">
-            <parameters>$(find robotek)/config/my_controllers.yaml</parameters>
-            <parameters>$(find robotek)/config/gaz_ros2_ctl_use_sim.yaml</parameters>
+            <!--gazebo simuluje controller manager a komunikuje se samotnyma kontrolerama -->
+            <parameters>$(find autobot)/params/my_controllers.yaml</parameters>
+            <parameters>$(find autobot)/params/gz_sim_time.yaml</parameters>
         </plugin>
     </gazebo>
